Commit message: Implement hybrid low-battery return-to-dock
- Add Scout-local battery dock guard with battery monitoring, guard state/control topics, vendor /nav_low_bat fallback, status monitoring, timeout, and retry handling.

- Add companion map-return controller that claims low-battery return only when localization, move_base, fresh pose, and the dock approach waypoint are healthy.

- Route normal navigation through the Scout safety filter and block planner commands during battery guard return, vendor docking, failed, and charging modes.

- Add runtime config, site defaults, launch wiring, install targets, URDF sensor frames, and live probe/validator checks for sensor, safety, and docking surfaces.

- Update README, setup, quickstart, validation, architecture notes, and checklist for the hybrid dock workflow and safe staging guidance.

- Add unit coverage for battery guard transitions, companion map-return eligibility, safety-filter battery modes, live probing, and validation contracts.

File: urdf/scout.urdf (robot description, URDF)
Before this commit: robot scout, 4 links, 3 joints
Links:
- added link tof_link, mass 0.001; visual box size=0.01 0.01 0.01
Joints:
- added joint base_to_tof: type fixed, parent base_link, child tof_link, origin xyz=0.075 0 0.04 rpy=0 0 0
